Commit message: SomethingProblem-221028

File: urdf/spmr02.urdf (robot description, URDF)
Before this commit: robot spmr02, 5 links, 4 joints
Joints:
- joint left_wheel_joint: axis -1 0 0 -> 1 0 0
- joint right_wheel_joint: axis 1 0 0 -> -1 0 0

Commit message: EditingURDF-2nd-221028

File: urdf/spmr02.urdf (robot description, URDF)
Before this commit: robot spmr02, 5 links, 4 joints
Links:
- link right_wheel_link: geometry collision mesh filename=package://spmr02/meshes/right_wheel_link.STL; visual mesh filename=filename=package://spmr02/meshes/right_wheel_link.STL
Joints:
- joint left_wheel_joint: origin xyz=0 -0.40407 -0.001 rpy=1.5708 0 1.5708 -> xyz=0 -0.40407 0 rpy=1.5708 0 1.5708
- joint right_wheel_joint: axis -1 0 0 -> 1 0 0; origin xyz=0 0.40407 -0.001 rpy=1.5708 0 -1.5708 -> xyz=0 0.40407 0 rpy=1.5708 0 -1.5708

Commit message: EditingURDF-please-221029

File: urdf/spmr02.urdf (robot description, URDF)
Before this commit: robot spmr02, 5 links, 4 joints
Links:
- link LR_scan_link: mass 1 -> 0.0083364
- link RF_scan_link: mass 1 -> 0.0083364
- link base_link: mass 50 -> 37.767
- link right_wheel_link: geometry collision mesh filename=package://spmr02/meshes/right_wheel_link.STL; visual mesh filename=package://spmr02/meshes/right_wheel_link.STL

Commit message: EditingDone-221029

File: urdf/spmr02.urdf (robot description, URDF)
Before this commit: robot spmr02, 5 links, 4 joints
Joints:
- joint left_wheel_joint: origin xyz=0 -0.40407 0 rpy=1.5708 0 1.5708 -> xyz=0 -0.40407 -0.001 rpy=1.5708 0 1.5708
- joint right_wheel_joint: axis 1 0 0 -> -1 0 0; origin xyz=0 0.40407 0 rpy=1.5708 0 -1.5708 -> xyz=0 0.40407 -0.001 rpy=1.5708 0 -1.5708

Commit message: Editing_joint-state-publisher_221031

File: urdf/spmr02.urdf (robot description, URDF)
Before this commit: robot spmr02, 5 links, 4 joints
Links:
- link LR_scan_link: mass 1 -> 0.0083364
- link RF_scan_link: mass 1 -> 0.0083364
- link base_link: mass 50 -> 37.767
Joints:
- joint left_wheel_joint: axis -1 0 0 -> 1 0 0
- joint right_wheel_joint: axis 1 0 0 -> -1 0 0

Commit message: WehaveProblemThatIsLidarDirection-221031

File: urdf/spmr02.urdf (robot description, URDF)
Before this commit: robot spmr02, 5 links, 4 joints
Links:
- link LR_scan_link: mass 0.0083364 -> 0.008
- link RF_scan_link: mass 0.0083364 -> 0.008

Commit message: IllCheckRayPose-221101

File: urdf/spmr02.urdf (robot description, URDF)
Before this commit: robot spmr02, 5 links, 4 joints
Links:
- link base_link: mass 37.767 -> 50
Joints:
- joint LR_scan_joint: origin xyz=0.61848 -0.45171 -0.10141 rpy=-1.5708 0 -2.3562 -> xyz=0 0 0 rpy=0 0 0
- joint RF_scan_joint: origin xyz=-0.63018 0.50694 -0.10141 rpy=-1.5708 0 0.7854 -> xyz=0 0 0 rpy=0 0 0

Commit message: 221103_gmapping_ing

File: urdf/spmr02.urdf (robot description, URDF)
Before this commit: robot spmr02, 5 links, 4 joints
Links:
- link LR_scan_link: mass 0.0083364 -> 0.008; geometry visual mesh filename=package://spmr02/meshes/LR_scan_link.STL
- link RF_scan_link: mass 0.0083364 -> 0.008; geometry visual mesh filename=package://spmr02/meshes/RF_scan_link.STL
- link base_link: mass 37.767 -> 50
Joints:
- joint LR_scan_joint: origin xyz=0.61848 -0.45171 -0.10141 rpy=-1.5708 0 -2.3562 -> xyz=-0.60802 0.48579 -0.07 rpy=0 0 3.141592
- joint RF_scan_joint: origin xyz=-0.63018 0.50694 -0.10141 rpy=-1.5708 0 0.7854 -> xyz=0.60802 -0.48579 -0.07 rpy=0 0 0

Commit message: 221105_slam_ing

File: urdf/spmr02.urdf (robot description, URDF)
Before this commit: robot spmr02, 5 links, 4 joints
Joints:
- joint LR_scan_joint: axis 0 0 0 -> (none); origin xyz=-0.60802 0.48579 -0.07 rpy=0 0 3.141592 -> xyz=-0.60802 0.48579 -0.08 rpy=0 0 2.3561
- joint RF_scan_joint: axis 0 0 0 -> (none); origin xyz=0.60802 -0.48579 -0.07 rpy=0 0 0 -> xyz=0.60802 -0.48579 -0.08 rpy=0 0 -0.7853

Commit message: 221225_modify

File: urdf/spmr02.urdf (robot description, URDF)
Before this commit: robot spmr02, 5 links, 4 joints
Links:
- link LR_scan_link: mass 1 -> 0.008; geometry visual mesh filename=package://spmr02/meshes/LR_scan_link.STL
- link RF_scan_link: mass 1 -> 0.008; geometry visual mesh filename=package://spmr02/meshes/RF_scan_link.STL
Joints:
- joint LR_scan_joint: axis 0 0 0 -> (none); origin xyz=0.61848 -0.45171 -0.10141 rpy=-1.5708 0 -2.3562 -> xyz=-0.60802 0.48579 -0.08 rpy=0 0 2.3561
- joint RF_scan_joint: axis 0 0 0 -> (none); origin xyz=-0.63018 0.50694 -0.10141 rpy=-1.5708 0 0.7854 -> xyz=0.60802 -0.48579 -0.08 rpy=0 0 -0.7853
- joint left_wheel_joint: axis -1 0 0 -> 1 0 0
- joint right_wheel_joint: axis 1 0 0 -> -1 0 0

Commit message: gui

File: urdf/spmr02.urdf (robot description, URDF)
Before this commit: robot spmr02, 5 links, 4 joints
Links:
- added link L_camera, mass 0.046733; visual mesh filename=package://spmr02/meshes/L_camera.STL
- added link R_camera, mass 0.046733; visual mesh filename=package://spmr02/meshes/R_camera.STL
- link LR_scan_link: mass 1 -> 0.008; geometry visual mesh filename=package://spmr02/meshes/LR_scan_link.STL
- link RF_scan_link: mass 1 -> 0.008; geometry visual mesh filename=package://spmr02/meshes/RF_scan_link.STL
Joints:
- added joint L_camera-joint: type fixed, parent base_link, child L_camera, origin xyz=0 0.6595 0.19 rpy=-3.1416 1.5708 3.1416, axis 0 0 0
- added joint R_camera-joint: type fixed, parent base_link, child R_camera, origin xyz=0 -0.6595 0.19 rpy=-3.1416 1.5708 3.1416, axis 0 0 0
- joint LR_scan_joint: axis 0 0 0 -> (none); origin xyz=0.61848 -0.45171 -0.10141 rpy=-1.5708 0 -2.3562 -> xyz=-0.60802 0.48579 -0.08 rpy=0 0 2.3561
- joint RF_scan_joint: axis 0 0 0 -> (none); origin xyz=-0.63018 0.50694 -0.10141 rpy=-1.5708 0 0.7854 -> xyz=0.60802 -0.48579 -0.08 rpy=0 0 -0.7853
- joint left_wheel_joint: axis -1 0 0 -> 1 0 0
- joint right_wheel_joint: axis 1 0 0 -> -1 0 0

Commit message: ros text

File: urdf/spmr02.urdf (robot description, URDF)
Before this commit: robot spmr02, 5 links, 4 joints
Links:
- added link L_camera, mass 0.046733; visual mesh filename=package://spmr02/meshes/L_camera.STL
- added link R_camera, mass 0.046733; visual mesh filename=package://spmr02/meshes/R_camera.STL
- link LR_scan_link: geometry visual mesh filename=package://spmr02/meshes/LR_scan_link.STL
- link RF_scan_link: geometry visual mesh filename=package://spmr02/meshes/RF_scan_link.STL
Joints:
- added joint L_camera-joint: type fixed, parent base_link, child L_camera, origin xyz=0 -0.6595 0.19 rpy=-3.1416 1.5708 3.1416, axis 0 0 0
- added joint R_camera-joint: type fixed, parent base_link, child R_camera, origin xyz=0 0.6595 0.19 rpy=-3.1416 1.5708 3.1416, axis 0 0 0
- joint LR_scan_joint: axis 0 0 0 -> (none); origin xyz=0 0 0 rpy=0 0 0 -> xyz=-0.60802 0.48579 -0.08 rpy=0 0 2.3561
- joint RF_scan_joint: axis 0 0 0 -> (none); origin xyz=0 0 0 rpy=0 0 0 -> xyz=0.60802 -0.48579 -0.08 rpy=0 0 -0.7853
